File: r60.kicad_pcb (KiCad board)
At the start: 2 copper layers, 142 parts, among them K0 K_ESC, K0A1 K_0, K0B1 K_MIN, K0C1 K_EQL, K0D1 K_BS, K1 K_1, K10 K_TAB, K11 K_Q, K12 K_W, K13 K_E, K14 K_R, K15 K_T, K16 K_Y, K17 K_U, K18 K_I, K19 K_O, K1A1 K_P, K1B1 K_OBR, K1C1 K_CBR, K1D1 K_BSL, K2 K_2, K20 K_CAP, K21 K_A, K22 K_S, K23 K_D, K24 K_F, K25 K_G, K26 K_H, K27 K_J, K28 K_K, K29 K_L, K2A1 K_COL, K2B1 K_QOT, K2C1 K_ENT, K3 K_3, K30 K_LSH, K31 K_Z, K32 K_X, K33 K_C, K34 K_V, K35 K_B, K36 K_N, K37 K_M, K38 K_COM, K39 K_DOT, K3A1 K_QUE, K3B1 K_RSH, K4 K_4, K40 K_LCL, K41 K_LWN, K42 K_LAL, K44 K_LSP, K45 K_RSP, K47 K_RAL, K48 K_LFT, K49 K_RT, K4A1 K_UP, K4B1 K_DWN, K5 K_5, K6 K_6, K7 K_7, K8 K_8, K9 K_9, P1 USB_B, SW1 SW_Push, U1 ATmega32U4-AU, Y1 16MHz

Commit message: layout board outlines and mounting holes
Parts:
- added REF**: MountingHole_2.7mm_M2.5, Mounting_Holes:MountingHole_2.7mm_M2.5, F.Cu at (54.8, 71.4)
- added REF**: MountingHole_2.7mm_M2.5, Mounting_Holes:MountingHole_2.7mm_M2.5, F.Cu at (157.2, 90.5)
- added REF**: MountingHole_2.7mm_M2.5, Mounting_Holes:MountingHole_2.7mm_M2.5, F.Cu at (290.5, 71.4)
- added REF**: MountingHole_2.7mm_M2.5, Mounting_Holes:MountingHole_2.7mm_M2.5, F.Cu at (219.1, 128.6)
- added REF**: MountingHole_2.7mm_M2.5, Mounting_Holes:MountingHole_2.7mm_M2.5, F.Cu at (28.6, 100.0)
- added REF**: MountingHole_2.7mm_M2.5, Mounting_Holes:MountingHole_2.7mm_M2.5, F.Cu at (314.3, 100.0)
- moved C2 161.0 mm to (35.7, 104.8), turned to 270 degrees
- moved Y1 149.5 mm to (40.5, 107.2)
- moved C1 136.1 mm to (45.2, 104.8), turned to 270 degrees
- moved C8 131.3 mm to (31.0, 119.1), turned to 270 degrees
- moved R4 99.2 mm to (52.4, 119.1)
- moved R3 97.7 mm to (57.1, 97.6)
- moved SW1 67.1 mm to (57.1, 90.5), turned to 270 degrees
- moved P1 32.8 mm to (47.6, 47.0)
- moved R1 32.3 mm to (48.9, 56.6), turned to 270 degrees
- moved R2 26.8 mm to (46.3, 56.6), turned to 90 degrees
- moved C5 12.8 mm to (35.7, 128.6)
- moved D1 10.1 mm to (57.1, 47.6), turned to 180 degrees
- moved D0 10.1 mm to (38.1, 47.6), turned to 180 degrees
- moved D44 10.1 mm to (138.1, 123.8)
- moved D45 10.1 mm to (176.2, 123.8)
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Other:
- board outline added: 285.8 x 95.3 mm

Commit message: finish first pass of routing board
Parts:
- moved C8 11.5 mm to (33.7, 130.2)
- moved D16 8.80 mm to (159.5, 67.7), turned to 270 degrees
- moved D1B1 8.80 mm to (254.8, 67.7), turned to 270 degrees
- moved D1C1 8.80 mm to (273.8, 67.7), turned to 270 degrees
- moved D1D1 8.80 mm to (297.7, 67.7), turned to 270 degrees
- moved D13 8.80 mm to (102.4, 67.7), turned to 270 degrees
- moved D14 8.80 mm to (121.4, 67.7), turned to 270 degrees
- moved D10 8.80 mm to (40.5, 67.7), turned to 270 degrees
- moved D11 8.80 mm to (64.3, 67.7), turned to 270 degrees
- moved D12 8.80 mm to (83.3, 67.7), turned to 270 degrees
- moved D15 8.80 mm to (140.5, 67.7), turned to 270 degrees
- moved D17 8.80 mm to (178.6, 67.7), turned to 270 degrees
- moved D18 8.80 mm to (197.6, 67.7), turned to 270 degrees
- moved D19 8.80 mm to (216.7, 67.7), turned to 270 degrees
- moved D1A1 8.80 mm to (235.7, 67.7), turned to 270 degrees
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Connections:
- K42 pad 2: (no net) -> /C2
Routing:
- net /R0: track 0.00 -> 339.1 mm, vias 0 -> 2
- net /C11: track 0.00 -> 332.1 mm, vias 0 -> 2
- net /C12: track 0.00 -> 319.2 mm, vias 0 -> 2
- net /C13: track 0.00 -> 318.7 mm, vias 0 -> 4
- net /C8: track 0.00 -> 318.5 mm, vias 0 -> 4
- net /R1: track 0.00 -> 316.1 mm, vias 0 -> 2
- net /C10: track 0.00 -> 313.1 mm, vias 0 -> 2
- net /C9: track 0.00 -> 299.7 mm, vias 0 -> 1
- net /R2: track 0.00 -> 289.4 mm, vias 0 -> 2
- net /C7: track 0.00 -> 287.9 mm, vias 0 -> 4
- net /R4: track 0.00 -> 245.5 mm, vias 0 -> 2
- net /C5: track 0.00 -> 240.5 mm, vias 0 -> 2
- net /R3: track 0.00 -> 237.2 mm, vias 0 -> 2
- net /C6: track 0.00 -> 204.4 mm
- net /C4: track 0.00 -> 185.7 mm, vias 0 -> 1
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- added copper zone on B.Cu, net GND
- added copper zone on F.Cu, net GND

Commit message: final layout for rev a
Parts:
- REF** (x6): value MountingHole_2.7mm_M2.5 -> (none)
- moved REF** 0.89 mm to (289.6, 71.4)
Other:
- board text added: "r60 rev A Ron Pedde <ron@pedde.com> github.com/rpedde/r60"
Changed lines of the file:
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@@
     (links 234)
     (no_connects 0)
-    (area 28.499999 42.787499 314.400001 138.187501)
+    (area 22.025 41.274999 320.875 138.261701)
     (thickness 1.6)
-    (drawings 8)
+    (drawings 9)
     (tracks 905)
     (zones 0)
@@
     (visible_elements FFFFFF7F)
     (pcbplotparams
-      (layerselection 0x00030_80000001)
-      (usegerberextensions false)
+      (layerselection 0x010f0_80000001)
+      (usegerberextensions true)
       (excludeedgelayer true)
       (linewidth 0.100000)
@@
       (outputformat 1)
       (mirror false)
-      (drillshape 1)
+      (drillshape 0)
       (scaleselection 1)
-      (outputdirectory ""))
+      (outputdirectory gerber/))
   )
   (net 0 "")
@@
       (effects (font (size 1 1) (thickness 0.15)))
     )
-    (fp_text value MountingHole_2.7mm_M2.5 (at 0 3.7) (layer F.Fab)
+    (fp_text value "" (at 0 3.7) (layer F.Fab)
       (effects (font (size 1 1) (thickness 0.15)))
     )
@@
       (effects (font (size 1 1) (thickness 0.15)))
     )
-    (fp_text value MountingHole_2.7mm_M2.5 (at 0 3.7) (layer F.Fab)
+    (fp_text value "" (at 0 3.7) (layer F.Fab)
       (effects (font (size 1 1) (thickness 0.15)))
     )
     (fp_circle (center 0 0) (end 2.7 0) (layer Cmts.User) (width 0.15))
     (fp_circle (center 0 0) (end 2.95 0) (layer F.CrtYd) (width 0.05))
-    (pad 1 thru_hole circle (at 0 0) (size 7 7) (drill oval 5.2 2.7) (layers *.Cu *.Mask))
+    (pad 3 thru_hole circle (at 0 0) (size 7 7) (drill oval 5.2 2.7) (layers *.Cu *.Mask))
   )
   (module Mounting_Holes:MountingHole_2.7mm_M2.5 (layer F.Cu)
-    (at 290.5125 71.4375)
+    (at 289.6225 71.4375)
     (descr "Mounting Hole 2.7mm, no annular, M2.5")
     (tags "mounting hole 2.7mm no annular m2.5")
@@
       (effects (font (size 1 1) (thickness 0.15)))
     )
-    (fp_text value MountingHole_2.7mm_M2.5 (at 0 3.7) (layer F.Fab)
+    (fp_text value "" (at 0 3.7) (layer F.Fab)
       (effects (font (size 1 1) (thickness 0.15)))
     )
     (fp_circle (center 0 0) (end 2.7 0) (layer Cmts.User) (width 0.15))
     (fp_circle (center 0 0) (end 2.95 0) (layer F.CrtYd) (width 0.05))
-    (pad 1 thru_hole circle (at 0 0) (size 7 7) (drill oval 5.2 2.7) (layers *.Cu *.Mask))
+    (pad 5 thru_hole circle (at 0 0) (size 7 7) (drill oval 5.2 2.7) (layers *.Cu *.Mask))
   )
   (module Mounting_Holes:MountingHole_2.7mm_M2.5 (layer F.Cu)
@@
       (effects (font (size 1 1) (thickness 0.15)))
     )
-    (fp_text value MountingHole_2.7mm_M2.5 (at 0 3.7) (layer F.Fab)
+    (fp_text value "" (at 0 3.7) (layer F.Fab)
       (effects (font (size 1 1) (thickness 0.15)))
     )
     (fp_circle (center 0 0) (end 2.7 0) (layer Cmts.User) (width 0.15))
     (fp_circle (center 0 0) (end 2.95 0) (layer F.CrtYd) (width 0.05))
-    (pad 1 thru_hole circle (at 0 0) (size 7 7) (drill oval 5.2 2.7) (layers *.Cu *.Mask))
+    (pad 4 thru_hole circle (at 0 0) (size 7 7) (drill oval 5.2 2.7) (layers *.Cu *.Mask))
   )
   (module Mounting_Holes:MountingHole_2.7mm_M2.5 (layer F.Cu)
@@
       (effects (font (size 1 1) (thickness 0.15)))
     )
-    (fp_text value MountingHole_2.7mm_M2.5 (at 0 3.7) (layer F.Fab)
+    (fp_text value "" (at 0 3.7) (layer F.Fab)
       (effects (font (size 1 1) (thickness 0.15)))
     )
     (fp_circle (center 0 0) (end 2.7 0) (layer Cmts.User) (width 0.15))
     (fp_circle (center 0 0) (end 2.95 0) (layer F.CrtYd) (width 0.05))
-    (pad 1 thru_hole oval (at 0 0) (size 12.7 5) (drill oval 10 2.7) (layers *.Cu *.Mask))
+    (pad 2 thru_hole oval (at 0 0) (size 12.7 5) (drill oval 10 2.7) (layers *.Cu *.Mask))
   )
   (module Mounting_Holes:MountingHole_2.7mm_M2.5 (layer F.Cu)
@@
       (effects (font (size 1 1) (thickness 0.15)))
     )
-    (fp_text value MountingHole_2.7mm_M2.5 (at 0 3.7) (layer F.Fab)
+    (fp_text value "" (at 0 3.7) (layer F.Fab)
       (effects (font (size 1 1) (thickness 0.15)))
     )
     (fp_circle (center 0 0) (end 2.7 0) (layer Cmts.User) (width 0.15))
     (fp_circle (center 0 0) (end 2.95 0) (layer F.CrtYd) (width 0.05))
-    (pad 1 thru_hole oval (at 0 0) (size 12.7 5) (drill oval 10 2.7) (layers *.Cu *.Mask))
+    (pad 6 thru_hole oval (at 0 0) (size 12.7 5) (drill oval 10 2.7) (layers *.Cu *.Mask))
+  )
+  (gr_text "r60 rev A\nRon Pedde <ron@pedde.com>\ngithub.com/rpedde/r60" (at 300.355 101.2825 90) (layer B.SilkS)
+    (effects (font (size 1.5 1.5) (thickness 0.3)) (justify left mirror))
   )
   (gr_line (start 311.94375 138.1125) (end 30.95625 138.1125) (angle 90) (layer Edge.Cuts) (width 0.15))
@@
   (segment (start 46.94025 124.3965) (end 48.861 124.3965) (width 0.3) (layer B.Cu) (net 93))
   (segment (start 48.861 124.3965) (end 49.911 124.3965) (width 0.3) (layer B.Cu) (net 93))
-  (zone (net 1) (net_name GND) (layer F.Cu) (hatch edge 0.508)
-    (connect_pads (clearance 0.508))
-    (min_thickness 0.254)
-    (fill yes (arc_segments 16) (thermal_gap 0.508) (thermal_bridge_width 0.508))
-    (polygon
-      (pts
-        (xy 28.575 42.8625) (xy 314.325 42.8625) (xy 314.325 138.1125) (xy 28.575 138.1125) (xy 28.575 45.24375)
-      )
-    )
-  )
   (zone (net 1) (net_name GND) (layer B.Cu) (hatch edge 0.508)
     (connect_pads (clearance 0.508))
